File: HACK CLUB RELATED.kicad_pcb (KiCad board)
At the start: 4 copper layers, 88 x 155 mm, 104 parts, among them CN3 KH-FG0.5-H2.0-40PIN, J1 Battery_JST_PH2, J2 Conn_01x02, J3 Conn_01x03, J4 Conn_01x03, J5 Conn_01x03, Q1 LBSS138LT1G, Q2 AO3407A, SW1 SW_Push, SW2 SW_Push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

Commit message: Fix gitignore filename
Routing:
- net +5V: track 392.7 -> 403.8 mm
- net (no net): track 0.00 -> 1.21 mm, vias 0 -> 1
Changed lines of the file:
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@@
 	)
 	(segment
+		(start 115.5 142.25)
+		(end 115.5 141.75)
+		(width 0.2)
+		(layer "F.Cu")
+		(net 0)
+	)
+	(segment
+		(start 115 142.75)
+		(end 115.5 142.25)
+		(width 0.2)
+		(layer "F.Cu")
+		(net 0)
+	)
+	(via
+		(at 115.5 141.75)
+		(size 0.6)
+		(drill 0.3)
+		(layers "F.Cu" "B.Cu")
+		(net 0)
+	)
+	(segment
 		(start 111.05 130.151)
 		(end 111.05 129.5)
@@
 	)
 	(segment
+		(start 108.5498 121.75)
+		(end 108.5999 121.8001)
+		(width 0.5)
+		(layer "F.Cu")
+		(net 8)
+	)
+	(segment
+		(start 107.05 129.6905)
+		(end 106.8405 129.6905)
+		(width 0.1998)
+		(layer "F.Cu")
+		(net 8)
+	)
+	(segment
+		(start 105.6491 125.016)
+		(end 105.9811 125.016)
+		(width 0.5)
+		(layer "F.Cu")
+		(net 8)
+	)
+	(segment
 		(start 82.5983 172.8)
 		(end 82.5983 174.7)
@@
 	)
 	(segment
+		(start 108.5999 128.8483)
+		(end 108.5017 128.8483)
+		(width 0.1998)
+		(layer "F.Cu")
+		(net 8)
+	)
+	(segment
+		(start 106.8405 129.6905)
+		(end 106.65 129.5)
+		(width 0.1998)
+		(layer "F.Cu")
+		(net 8)
+	)
+	(segment
 		(start 151.75 109)
 		(end 150.5863 109)
@@
 	)
 	(segment
+		(start 108.5498 121.75)
+		(end 108.5498 122.4473)
+		(width 0.5)
+		(layer "F.Cu")
+		(net 8)
+	)
+	(segment
 		(start 108.5999 128.8483)
 		(end 108.5375 128.9107)
@@
 	)
 	(segment
-		(start 107.05 129.6905)
-		(end 107.05 130.1016)
-		(width 0.1998)
-		(layer "F.Cu")
-		(net 8)
-	)
-	(segment
 		(start 81.3494 117.8497)
 		(end 81.3494 118.25)
@@
 	)
 	(segment
-		(start 106.65 129.5)
-		(end 106.65 130.1016)
-		(width 0.1998)
-		(layer "F.Cu")
-		(net 8)
-	)
-	(segment
 		(start 108.5375 128.9107)
 		(end 108.5375 129.5)
@@
 	)
 	(segment
+		(start 108.5017 128.8483)
+		(end 107.85 129.5)
+		(width 0.1998)
+		(layer "F.Cu")
+		(net 8)
+	)
+	(segment
 		(start 77.8555 123.5)
 		(end 77.77 123.5)
@@
 	)
 	(segment
+		(start 108.5999 121.8001)
+		(end 108.5999 128.8483)
+		(width 0.5)
+		(layer "F.Cu")
+		(net 8)
+	)
+	(segment
 		(start 81.3494 121.9506)
 		(end 80.3 123)
@@
 	)
 	(segment
-		(start 107.05 130.1016)
-		(end 106.65 130.1016)
-		(width 0.1998)
-		(layer "F.Cu")
-		(net 8)
-	)
-	(segment
 		(start 114.8957 133.3916)
 		(end 115.05 133.2373)
@@
 	)
 	(segment
+		(start 105.9811 125.016)
+		(end 108.5498 122.4473)
+		(width 0.5)
+		(layer "F.Cu")
+		(net 8)
+	)
+	(segment
 		(start 88.77 170.75)
 		(end 88.77 171.5216)
@@
 	(segment
 		(start 108.5498 116.1882)
-		(end 108.5498 122.4473)
+		(end 108.5498 121.75)
 		(width 0.5)
 		(layer "F.Cu")
