File: KiCAD files/HACK CLUB RELATED.kicad_pcb (KiCad board)
At the start: 4 copper layers, 88 x 155 mm, 104 parts, among them CN3 KH-FG0.5-H2.0-40PIN, J1 Battery_JST_PH2, J2 Conn_01x02, J3 Conn_01x03, J4 Conn_01x03, J5 Conn_01x03, Q1 LBSS138LT1G, Q2 AO3407A, SW1 SW_Push, SW2 SW_Push, SW3 SW_Push, U1 BQ25895RTW, U2 TPS61235PRWLR, U3 FUSB302BMPX, U4 SGM2036-3.3YN5G/TR, U5 SGM2036-1.8YN5G/TR, U6 MAX98357AETE+T

Commit message: Add CAD assembly and enclosures
Parts:
- moved SW2 11.5 mm to (146.2, 56.8)
- moved C32 6.52 mm to (141.2, 52.2)
- moved SW3 4.25 mm to (146.2, 41.0)
Routing:
- net GND: track 173.3 -> 179.9 mm
- net GPIO_VOL_UP: track 138.5 -> 139.7 mm
- net GPIO_VOL_DN: track 124.3 -> 124.9 mm, vias 3 -> 4
Changed lines of the file:
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@@
 	(footprint "Button_Switch_THT:SW_PUSH_6mm_H5mm"
 		(layer "F.Cu")
-		(at 146.25 45.25)
+		(at 146.25 56.75)
 		(descr "tactile push button, 6x6mm e.g. PHAP33xx series, height=5mm")
 		(tags "tact sw push 6mm")
@@
 	(footprint "Capacitor_SMD:C_0402_1005Metric"
 		(layer "F.Cu")
-		(at 140.75 45.75 90)
+		(at 141.25 52.25 90)
 		(descr "Capacitor SMD 0402 (1005 Metric), square (rectangular) end terminal, IPC-7351 nominal, (Body size source: IPC-SM-782 page 76, https://www.pcb-3d.com/wordpress/wp-content/uploads/ipc-sm-782a_amendment_1_and_2.pdf), generated with kicad-footprint-generator")
 		(tags "capacitor")
@@
 	(footprint "Button_Switch_THT:SW_PUSH_6mm_H5mm"
 		(layer "F.Cu")
-		(at 146.25 36.75)
+		(at 146.25 41)
 		(descr "tactile push button, 6x6mm e.g. PHAP33xx series, height=5mm")
 		(tags "tact sw push 6mm")
@@
 	)
 	(segment
+		(start 146.23 45.27)
+		(end 146.25 45.25)
+		(width 0.2)
+		(layer "F.Cu")
+		(net 1)
+	)
+	(segment
 		(start 75.25 121.409432)
 		(end 75.225973 121.433459)
@@
 	)
 	(segment
+		(start 152.75 45.25)
+		(end 146.25 45.25)
+		(width 0.2)
+		(layer "B.Cu")
+		(net 1)
+	)
+	(segment
 		(start 93 109.75)
 		(end 90.25 109.75)
@@
 	)
 	(segment
-		(start 146.23 45.27)
-		(end 146.25 45.25)
-		(width 0.2)
-		(layer "F.Cu")
-		(net 17)
-	)
-	(segment
 		(start 121.5648 127.7247)
 		(end 121.9675 128.1274)
@@
 	)
 	(segment
+		(start 146.25 56.75)
+		(end 146.875 56.125)
+		(width 0.2)
+		(layer "F.Cu")
+		(net 17)
+	)
+	(segment
+		(start 141.25 50)
+		(end 141.25 51.77)
+		(width 0.2)
+		(layer "F.Cu")
+		(net 17)
+	)
+	(segment
 		(start 121.926 124.564)
 		(end 121.926 49.0743)
@@
 	)
 	(segment
+		(start 141.25 51.77)
+		(end 142.52 51.77)
+		(width 0.2)
+		(layer "F.Cu")
+		(net 17)
+	)
+	(segment
+		(start 147.5 56.75)
+		(end 154 56.75)
+		(width 0.2)
+		(layer "F.Cu")
+		(net 17)
+	)
+	(segment
 		(start 121.5648 125.25)
 		(end 121.5648 127.7247)
@@
 	)
 	(segment
-		(start 118.170481 130.084919)
-		(end 118.25 130.0054)
+		(start 146.875 56.125)
+		(end 147.5 56.75)
 		(width 0.2)
 		(layer "F.Cu")
@@
 	)
 	(segment
-		(start 140.75 45.27)
-		(end 146.23 45.27)
+		(start 118.170481 130.084919)
+		(end 118.25 130.0054)
 		(width 0.2)
 		(layer "F.Cu")
@@
 		(net 17)
 	)
+	(segment
+		(start 142.52 51.77)
+		(end 146.875 56.125)
+		(width 0.2)
+		(layer "F.Cu")
+		(net 17)
+	)
 	(via
 		(at 121.9675 128.1274)
@@
 		(net 17)
 	)
+	(via
+		(at 141.25 50)
+		(size 0.6)
+		(drill 0.3)
+		(layers "F.Cu" "B.Cu")
+		(net 17)
+	)
 	(segment
 		(start 117.751978 130.039055)
@@
 	)
 	(segment
-		(start 125.7503 45.25)
-		(end 123.4625 47.5378)
-		(width 0.2)
-		(layer "B.Cu")
-		(net 17)
-	)
-	(segment
 		(start 117.751978 129.814122)
 		(end 119.4387 128.1274)
@@
 	)
 	(segment
-		(start 146.25 45.25)
-		(end 125.7503 45.25)
+		(start 123.4625 47.5378)
+		(end 138.7878 47.5378)
 		(width 0.2)
 		(layer "B.Cu")
@@
 	)
 	(segment
-		(start 152.75 45.25)
-		(end 146.25 45.25)
+		(start 138.7878 47.5378)
+		(end 141.25 50)
 		(width 0.2)
 		(layer "B.Cu")
@@
 	)
 	(segment
+		(start 140.1605 41)
+		(end 140.1605 70.4933)
+		(width 0.2)
+		(layer "F.Cu")
+		(net 18)
+	)
+	(segment
 		(start 143.5479 123.915176)
 		(end 137.613738 129.849338)
@@
 	(segment
 		(start 140.1605 40.366)
-		(end 140.1605 70.4933)
+		(end 140.1605 41)
+		(width 0.2)
+		(layer "F.Cu")
+		(net 18)
+	)
+	(segment
+		(start 146.25 41)
+		(end 152.75 41)
 		(width 0.2)
 		(layer "F.Cu")
@@
 	)
 	(segment
-		(start 141.3233 36.75)
-		(end 146.25 36.75)
+		(start 140.1605 41)
+		(end 146.25 41)
 		(width 0.2)
 		(layer "F.Cu")
@@
 		(net 18)
 	)
-	(segment
-		(start 146.25 36.75)
-		(end 152.75 36.75)
-		(width 0.2)
-		(layer "B.Cu")
-		(net 18)
-	)
